File: hardware/ac400.kicad_sch (KiCad schematic)
At the start: 71 parts, among them J1 AVR-ISP-10, J2 LOW OUT, J3 MID OUT, J4 HIGH OUT, J5 COMMON OUT, J6 COMMON IN, J7 LINE IN, J8 3.3V IN, K1 SRD-03VDC-SL-C, K2 SRD-03VDC-SL-C, K3 SRD-03VDC-SL-C, Q1 IRLML2502, Q2 IRLML2502, Q3 IRLML2502, Q4 IRLML2502, SW1 ON, SW2 OFF, U1 ATmega88PA-A, U2 TSOP38238

Commit message: "final" touches on v1 board
Parts:
- added SYM2: Julian7 logo, ac400:Julian7 maker's mark, symbol Graphic:Logo_Open_Hardware_Small
- C2: footprint PCM_Capacitor_THT_AKL:C_Radial_D8.0mm_H11.5mm_P3.50mm -> Capacitor_THT:CP_Radial_D8.0mm_P3.50mm
- D1, D2, D3: footprint Diode_SMD:D_0805_2012Metric_Pad1.15x1.40mm_HandSolder -> Diode_SMD:D_SOD-323
- J2, J3, J4, J5, J6, J7, J8, TP1, TP2, TP3, TP4: now left out of the parts list
- SYM1: now in the parts list
- TP5: renamed from TP6; now left out of the parts list
- TP6: renamed from TP5; now left out of the parts list
- TP7: renamed from TP8; now left out of the parts list
- TP8: renamed from TP7; now left out of the parts list
Connections:
- net LINE: no longer J2.1 (Pin_1), J3.1 (Pin_1), J4.1 (Pin_1), K1.3, K2.3, K3.3
- net Mid Drain: now reaches D2.2 (A), K2.2, Q2.3 (D), TP5.1
- net Low Drain: now reaches D1.2 (A), K1.2, Q1.3 (D), TP3.1
- net Buzz Drain: now reaches BZ1.2 (-), Q4.3 (D)
- removed net Mosfet gate: D3.2 (A), K3.2, Q1.1 (G), Q2.1 (G), Q3.3 (D), Q4.1 (G), R1.2, R17.2, R18.2, R2.2, R4.2, R5.2, TP4.1, TP6.1, TP7.1
- new net: Q2.1 (G), R4.2, R5.2, TP6.1
- new net: Q1.1 (G), R1.2, R2.2, TP4.1
- new net: Q4.1 (G), R17.2, R18.2
- new net HIGH OUT: J4.1 (Pin_1), K3.3
- new net High Drain: D3.2 (A), K3.2, Q3.3 (D), TP7.1
- new net LOW OUT: J2.1 (Pin_1), K1.3
- new net MID OUT: J3.1 (Pin_1), K2.3
Other:
- moved on the sheet: J2, J3, J4, K1, K2, K3, R3, R6, R9

Commit message: mounting holes distance and library references fix
Parts:
- J2, J3, J4, J5, J6, J7, J8, JP1, TP1, TP2, TP3, TP4, TP5, TP6, TP7, TP8: now in the parts list
- SYM1: footprint ac400:AC400 Board -> ac400:board_shape
- SYM2: footprint ac400:Julian7 maker's mark -> ac400:julian7_makers_mark
