File: hardware/ac400.kicad_sch (KiCad schematic)
At the start: 72 parts, among them J1 AVR-ISP-10, J2 LOW OUT, J3 MID OUT, J4 HIGH OUT, J5 COMMON OUT, J6 COMMON IN, J7 LINE IN, J8 3.3V IN, K1 SRD-03VDC-SL-C, K2 SRD-03VDC-SL-C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

Commit message: Exclude non-component items from BOM
Parts:
- J2, J3, J4, J5, J6, J7, JP1, SYM1, SYM2, TP1, TP2, TP3, TP4, TP5, TP6, TP7, TP8: now left out of the parts list
- R3, R6, R9: value 2.2 0.25W -> 2.2

Commit message: Replace MCU, fix SPI pins and footprint
Parts:
- J1: value AVR-ISP-10 -> AVR-ISP-6; footprint Connector_IDC:IDC-Header_2x05_P2.54mm_Vertical -> Connector_IDC:IDC-Header_2x03_P2.54mm_Vertical; symbol Connector:AVR-ISP-10 -> Connector:AVR-ISP-6
- U1: value ATmega88PA-A -> ATmega328P-A; symbol MCU_Microchip_ATmega:ATmega88PA-A -> MCU_Microchip_ATmega:ATmega328P-A; Distributor Link 1 https://www.digikey.hu/hu/products/detail/microchip-technol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 -> https://www.digikey.hu/en/products/detail/microchip-technol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; Distributor Link 2 https://hu.mouser.com/ProductDetail/Microchip-Technology/ATMEGA88PA-AU?qs=VXy%252BgAb0zZQ5AzLsp2xy0A%3D%3D -> https://hu.mouser.com/ProductDetail/Microchip-Technology/ATMEGA328P-AU?qs=K8BHR703ZXiCmmgp6%2FGNmQ%3D%3D; Distributor Link 3 https://www.hestore.hu/prod_10029337.html -> https://www.hestore.hu/prod_10032542.html
Connections:
- net GND: no longer J1.10 (GND), J1.4 (GND), J1.8 (GND)
- net MISO: now also J1.1 (MISO), U1.16 (PB4); no longer J1.9 (MISO), U1.15 (PB3)
- net MOSI: now also J1.4 (MOSI), U1.15 (PB3); no longer J1.1 (MOSI), U1.14 (PB2)
- net SCK: now also J1.3 (SCK), U1.17 (PB5); no longer J1.7 (SCK), U1.13 (PB1)

Commit message: update design to KiCad 10.0 version
Parts:
- added R19: 10k, PCM_Resistor_SMD_AKL:R_0805_2012Metric_Pad1.15x1.40mm_HandSolder, symbol Device:R_Small
- added R20: 1k, PCM_Resistor_SMD_AKL:R_0805_2012Metric_Pad1.15x1.40mm_HandSolder, symbol Device:R_Small
Connections:
- net +3.3V: now also R19.2
- net RESET: now also R19.1, R20.2; no longer J1.5 (~{RST})
- new net: J1.5 (~{RST}), R20.1
Other:
- moved on the sheet: JP1
